File: bare_mega_1284/bare_mega_1284.kicad_pcb (KiCad board)
At the start: 4 copper layers, 60.2 x 37.5 mm, 29 parts, among them CON1 302-S101, J1 USB4085-GF-A_REVB, U1 ATMEGA1284P-AU, U4 FT231XS-U, Y1 Crystal 16.MHZ

Commit message: v2
Parts:
- removed TP11, TP19, TP20, TP21, TP22, TP43: TestPoint, TestPoint:TestPoint_Pad_2.0x2.0mm
- added PA2_7-IN1: TestPoint, TestPoint:TestPoint_Pad_2.0x2.0mm, F.Cu at (153.3, 84.2)
- added PA4_13-OUT1: TestPoint, TestPoint:TestPoint_Pad_2.0x2.0mm, F.Cu at (143.4, 115.5)
- added PA5_16-OUT1: TestPoint, TestPoint:TestPoint_Pad_2.0x2.0mm, F.Cu at (157.2, 115.5)
- added PB3_14-OUT1: TestPoint, TestPoint:TestPoint_Pad_2.0x2.0mm, F.Cu at (150.3, 115.5)
- added PD6_18-OUT1: TestPoint, TestPoint:TestPoint_Pad_2.0x2.0mm, F.Cu at (164.2, 115.5)
- added PD7_20-OUT1: TestPoint, TestPoint:TestPoint_Pad_2.0x2.0mm, F.Cu at (171.1, 115.5)
- moved PB4_12-OUT1 33.4 mm to (136.6, 115.5), turned to 180 degrees
- moved PA0_2-IN1 23.8 mm to (134.6, 84.2)
- moved PA1_5-IN1 23.0 mm to (144.3, 84.2)
- renumbered TP37 to PA0_2-IN1, TP36 to PA1_5-IN1, TP34 to PA3_9-IN1, TP44 to PB4_12-OUT1
Connections:
- S1 pad 1: /RES -> unconnected-(S1-COM_1-Pad1)
- S1 pad 4: GND -> unconnected-(S1-NO_2-Pad4)
- U1 pad 10: /RXD -> /TXD
- U1 pad 11: Net-(U1-(PCINT26/RXD1/INT0)_PD2) -> unconnected-(U1-(PCINT26/RXD1/INT0)_PD2-Pad11)
- U1 pad 15: unconnected-(U1-(PCINT30/OC2B/ICP)_PD6-Pad15) -> Net-(U1-(PCINT30/OC2B/ICP)_PD6)
- U1 pad 16: unconnected-(U1-(PCINT31/OC2A)_PD7-Pad16) -> Net-(U1-(PCINT31/OC2A)_PD7)
- U1 pad 19: Net-(U1-(PCINT16/SCL)_PC0) -> unconnected-(U1-(PCINT16/SCL)_PC0-Pad19)
- U1 pad 20: Net-(U1-(PCINT17/SDA)_PC1) -> unconnected-(U1-(PCINT17/SDA)_PC1-Pad20)
- U1 pad 21: Net-(U1-(PCINT18/TCK)_PC2) -> unconnected-(U1-(PCINT18/TCK)_PC2-Pad21)
- U1 pad 22: Net-(U1-(PCINT19/TMS)_PC3) -> unconnected-(U1-(PCINT19/TMS)_PC3-Pad22)
- U1 pad 32: unconnected-(U1-PA5_(ADC5/PCINT5)-Pad32) -> Net-(U1-PA5_(ADC5/PCINT5))
- U1 pad 33: unconnected-(U1-PA4_(ADC4/PCINT4)-Pad33) -> Net-(U1-PA4_(ADC4/PCINT4))
- U1 pad 35: unconnected-(U1-PA2_(ADC2/PCINT2)-Pad35) -> Net-(U1-PA2_(ADC2/PCINT2))
- U1 pad 9: /TXD -> /RXD
- U4 pad 14: unconnected-(U4-~{RESET}#-Pad14) -> +5V
Routing:
- net Net-(U1-PA4_(ADC4/PCINT4)): track 0.00 -> 39.6 mm, vias 0 -> 2
- net Net-(U1-PB4_(SS/OC0B/PCINT12)): track 11.3 -> 44.2 mm, vias 0 -> 2
- net Net-(U1-PA5_(ADC5/PCINT5)): track 0.00 -> 27.2 mm, vias 0 -> 2
- net Net-(U1-(PCINT31/OC2A)_PD7): track 0.00 -> 23.8 mm, vias 0 -> 2
- net Net-(U1-PB3_(AIN1/OC0A/PCINT11)): track 10.0 -> 29.6 mm, vias 0 -> 2
- net Net-(U1-PA0_(ADC0/PCINT0)): track 10.1 -> 29.6 mm
- net Net-(U1-(PCINT30/OC2B/ICP)_PD6): track 0.00 -> 17.5 mm, vias 0 -> 2
- net Net-(U1-(PCINT19/TMS)_PC3): track 16.8 -> 0.00 mm
- net Net-(U1-(PCINT16/SCL)_PC0): track 14.5 -> 0.00 mm
- net Net-(U1-(PCINT26/RXD1/INT0)_PD2): track 14.2 -> 0.00 mm, vias 2 -> 0
- net Net-(U1-(PCINT18/TCK)_PC2): track 13.5 -> 0.00 mm
- net Net-(U1-(PCINT17/SDA)_PC1): track 11.5 -> 0.00 mm
- net Net-(U1-PA2_(ADC2/PCINT2)): track 0.00 -> 11.4 mm
- net Net-(U1-PA1_(ADC1/PCINT1)): track 14.8 -> 19.7 mm
- net /TXD: track 12.4 -> 14.7 mm
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Other:
- board text added: "BARE 1284 V2.0 8/08/25"
- board text removed: "BARE 1284 V1.0 7/20/25"
