File: bare_mega_1284/bare_mega_1284.kicad_sch (KiCad schematic)
At the start: 29 parts, among them CON1 302-S101, J1 USB4085-GF-A_REVB, U1 ATMEGA1284P-AU, U4 FT231XS-U, Y1 Crystal 16.MHZ

Commit message: v2
Parts:
- removed TP11, TP19, TP20, TP21, TP22, TP43: TestPoint, TestPoint:TestPoint_Pad_2.0x2.0mm, symbol Connector:TestPoint
- added PA2_7-IN1, PA4_13-OUT1, PA5_16-OUT1, PB3_14-OUT1, PD6_18-OUT1, PD7_20-OUT1: TestPoint, TestPoint:TestPoint_Pad_2.0x2.0mm, symbol Connector:TestPoint
- renumbered TP37 to PA0_2-IN1, TP36 to PA1_5-IN1, TP34 to PA3_9-IN1, TP44 to PB4_12-OUT1
Connections:
- net +5V: now also U4.14 (~{RESET}#)
- net GND: no longer S1.4 (NO_2)
- net RES: no longer S1.1 (COM_1)
- net RXD: now also U1.9 ((PCINT24/RXD0/T3)_PD0); no longer U1.10 ((PCINT25/TXD0)_PD1)
- net TXD: now also U1.10 ((PCINT25/TXD0)_PD1); no longer U1.9 ((PCINT24/RXD0/T3)_PD0)
- net at U1.43 (PB3_(AIN1/OC0A/PCINT11)): now also PB3_14-OUT1.1
- net at U1.15 ((PCINT30/OC2B/ICP)_PD6): now also PD6_18-OUT1.1
- net at U1.16 ((PCINT31/OC2A)_PD7): now also PD7_20-OUT1.1
- net at U1.32 (PA5_(ADC5/PCINT5)): now also PA5_16-OUT1.1
- net at U1.33 (PA4_(ADC4/PCINT4)): now also PA4_13-OUT1.1
- net at U1.35 (PA2_(ADC2/PCINT2)): now also PA2_7-IN1.1
- no-connect marks 16 -> 15
Other:
- moved on the sheet: C2, C4
